File: CM3+IO Board.sch (EAGLE design)
At the start: 102 parts, among them J1 10103594-0001LF, J4 10103594-0001LF, U1 PAM2306AYPKE, U3 AP2331W, X1 1376408-1_DDR2_2.5V, X2 52745-0890, X3 52745-2290, X4 52745-2290, X5 52745-2290, X6 52745-2290

Commit message: Fixed Some Mistakes in Schematic and added CM3 pinout
I've gone over all the cosmponents and found some mistakes and added some lables. Looks good, but I'd still benifit from some other eyes.

Also created a spreadsheet of all the CMIO3 pins and lables
Parts:
- removed J1: 10103594-0001LF, Connectors:10103594-0001LF
- removed JP1: (no value), pinhead:PINHD-1X3
- added J15: 10103594-0001LF, Connectors:10103594-0001LF
- added J16: (no value), Wurth_Elektronik_Electromechanic_Input-Output_Connectors_rev19d:693071020811
- C1, C10, C3: value (none) -> 47u
- C13, C14: value (none) -> 1u
- C23, C24: value (none) -> 4.7u
- J2: value (none) -> 10103594-0001LF; device Wurth_Elektronik_Electromechanic_Input-Output_Connectors_rev19d:693071020811 -> Connectors:10103594-0001LF
- J4: value 10103594-0001LF -> (none); device Connectors:10103594-0001LF -> pinhead:PINHD-1X3
- L1, L2: value (none) -> 4.7u 2A
- R1, R4, R6: value 0R -> 0R 1%
- R10: value (none) -> 100K 1%
- R12: value (none) -> 1K 1%
- R3: value 470R -> 470R 1%
- R30: value (none) -> 47K 1%
- R31: value (none) -> 0R 1%
- renumbered J7 to J14, MF-MSMF200 to F1
Connections:
- net +V: now also J16.VDD; no longer J2.VDD
- net GND: now also J15.5, J15.SHIELD, J16.GND, J16.VSS, J2.5, J2.SHIELD, J4.3, X2-7.S; no longer J1.5, J1.SHIELD, J2.GND, J2.VSS, J4.5, J4.SHIELD, JP1.3, X2-8.S
- net GPIO38: now also X1-64.1
- net N$1: now also J2.1; no longer J1.1
- net N$7: now also J4.2; no longer JP1.2
- net SDX_CLK: now also J16.CLK; no longer J2.CLK
- net SDX_CMD: now also J16.CMD; no longer J2.CMD
- net SDX_D0: now also J16.DAT0; no longer J2.DAT0
- net SDX_D1: now also J16.DAT1; no longer J2.DAT1
- net SDX_D2: now also J16.DAT2; no longer J2.DAT2
- net SDX_D3: now also J16.CD/DAT3; no longer J2.CD/DAT3
- net USBB_DM: now also J15.2; no longer J4.2
- net USBB_DP: now also J15.3; no longer J4.3
- net VBUSB: now also J15.1; no longer JP1.1
- net VC_TCK: now also X2-8.S; no longer X2-7.S
Other:
- note added: "3216"
- note added: "J7"
- note added: "MF-MSMF200"
- note removed: "J2"
- moved on the sheet: C4
